File: hardware/tempLoggerNG.sch (KiCad schematic (older format))
At the start: 29 parts, among them CON1 MR-AVR-ISP-6, CON2 USB-MINI-B, CON3 USB-MINI-B, CON4 USB-MINI-B, CON5 USB-MINI-B, CON6 USB-MINI-B, IC1 ATMEGA168A-A, Q1 MOS_N, Q2 MOS_N, Q3 MOS_N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

Commit message: commandline: limit readout rate to 0.15 to be on the safe side
Parts:
- C1, C10, C2, C3, C4, C5, C6, C7, C8: symbol C -> C-RESCUE-tempLoggerNG
- R1, R2, R3, R4, R5, R6: symbol R -> R-RESCUE-tempLoggerNG
- U2: symbol NCP1117ST33T3G -> NCP1117ST33T3G-RESCUE-tempLoggerNG
Changed lines of the file:
@@
 EESchema Schematic File Version 2
+LIBS:tempLoggerNG-rescue
 LIBS:power
 LIBS:device
@@
 $EndComp
 $Comp
-L C C5
+L C-RESCUE-tempLoggerNG C5
 U 1 1 5661A975
 P 3800 6150
@@
 $EndComp
 $Comp
-L C C6
+L C-RESCUE-tempLoggerNG C6
 U 1 1 5661A9EC
 P 4400 6150
@@
 Connection ~ 4400 5800
 $Comp
-L GND #PWR01
+L GND-RESCUE-tempLoggerNG #PWR01
 U 1 1 5661AA62
 P 3800 6450
@@
 $EndComp
 $Comp
-L GND #PWR02
+L GND-RESCUE-tempLoggerNG #PWR02
 U 1 1 5661AA83
 P 4400 6450
@@
 	4300 5450 2800 5450
 $Comp
-L +3.3V #PWR03
+L +3.3V-RESCUE-tempLoggerNG #PWR03
 U 1 1 5661B096
 P 3400 5850
@@
 $EndComp
 $Comp
-L R R1
+L R-RESCUE-tempLoggerNG R1
 U 1 1 5661B0FB
 P 3400 6150
@@
 Connection ~ 3250 6400
 $Comp
-L GND #PWR04
+L GND-RESCUE-tempLoggerNG #PWR04
 U 1 1 5661B212
 P 3950 4450
@@
 	4100 3950 4100 3900
 $Comp
-L NCP1117ST33T3G U2
+L NCP1117ST33T3G-RESCUE-tempLoggerNG U2
 U 1 1 5661B2D6
 P 1800 4150
@@
 $EndComp
 $Comp
-L +3.3V #PWR07
+L +3.3V-RESCUE-tempLoggerNG #PWR07
 U 1 1 5661B3CA
 P 2400 4000
@@
 $EndComp
 $Comp
-L C C3
+L C-RESCUE-tempLoggerNG C3
 U 1 1 5661B3F5
 P 1200 4300
@@
 $EndComp
 $Comp
-L C C4
+L C-RESCUE-tempLoggerNG C4
 U 1 1 5661B4E3
 P 2400 4300
@@
 $EndComp
 $Comp
-L GND #PWR08
+L GND-RESCUE-tempLoggerNG #PWR08
 U 1 1 5661B537
 P 1200 4600
@@
 $EndComp
 $Comp
-L GND #PWR09
+L GND-RESCUE-tempLoggerNG #PWR09
 U 1 1 5661B567
 P 1800 4600
@@
 $EndComp
 $Comp
-L GND #PWR010
+L GND-RESCUE-tempLoggerNG #PWR010
 U 1 1 5661B590
 P 2400 4600
@@
 $EndComp
 $Comp
-L R R4
+L R-RESCUE-tempLoggerNG R4
 U 1 1 5661B873
 P 5000 6800
@@
 $EndComp
 $Comp
-L R R3
+L R-RESCUE-tempLoggerNG R3
 U 1 1 5661B8F2
 P 5000 6650
@@
 	5400 6500 5400 6200
 $Comp
-L +3.3V #PWR012
+L +3.3V-RESCUE-tempLoggerNG #PWR012
 U 1 1 5661BBAD
 P 5250 6300
@@
 $EndComp
 $Comp
-L R R2
+L R-RESCUE-tempLoggerNG R2
 U 1 1 5661BBD4
 P 5000 6450
@@
 Connection ~ 4600 6650
 $Comp
-L GND #PWR013
+L GND-RESCUE-tempLoggerNG #PWR013
 U 1 1 5661BD86
 P 6700 7400
@@
 $EndComp
 $Comp
-L GND #PWR014
+L GND-RESCUE-tempLoggerNG #PWR014
 U 1 1 5661BDC2
 P 5300 7400
@@
 Connection ~ 6700 7100
 $Comp
-L GND #PWR015
+L GND-RESCUE-tempLoggerNG #PWR015
 U 1 1 5661C251
 P 650 7550
@@
 Connection ~ 650  7250
 $Comp
-L +3.3V #PWR016
+L +3.3V-RESCUE-tempLoggerNG #PWR016
 U 1 1 5661C405
 P 650 4850
@@
 	650  5250 900  5250
 $Comp
-L GND #PWR017
+L GND-RESCUE-tempLoggerNG #PWR017
 U 1 1 5661C539
 P 650 6050
@@
 $EndComp
 $Comp
-L GND #PWR018
+L GND-RESCUE-tempLoggerNG #PWR018
 U 1 1 5661C56E
 P 850 6050
@@
 $EndComp
 $Comp
-L C C2
+L C-RESCUE-tempLoggerNG C2
 U 1 1 5661C597
 P 850 5750
@@
 $EndComp
 $Comp
-L C C1
+L C-RESCUE-tempLoggerNG C1
 U 1 1 5661C638
 P 650 5750
@@
 	4050 6750 4050 6800
 $Comp
-L +3.3V #PWR019
+L +3.3V-RESCUE-tempLoggerNG #PWR019
 U 1 1 566203CC
 P 6050 1100
@@
 	6050 1150 6050 1100
 $Comp
-L GND #PWR020
+L GND-RESCUE-tempLoggerNG #PWR020
 U 1 1 566204F8
 P 6050 1250
@@
 	6600 1250 6050 1250
 $Comp
-L +3.3V #PWR021
+L +3.3V-RESCUE-tempLoggerNG #PWR021
 U 1 1 5662064B
 P 9300 1650
@@
 	9300 1750 9300 1650
 $Comp
-L GND #PWR022
+L GND-RESCUE-tempLoggerNG #PWR022
 U 1 1 56620738
 P 8850 1850
@@
 	8850 1850 8500 1850
 $Comp
-L C C10
+L C-RESCUE-tempLoggerNG C10
 U 1 1 566207C9
 P 9500 1750
@@
 $EndComp
 $Comp
-L GND #PWR023
+L GND-RESCUE-tempLoggerNG #PWR023
 U 1 1 56620827
 P 9850 1750
@@
 	9700 1750 9850 1750
 $Comp
-L C C7
+L C-RESCUE-tempLoggerNG C7
 U 1 1 56620970
 P 5850 1150
@@
 $EndComp
 $Comp
-L GND #PWR024
+L GND-RESCUE-tempLoggerNG #PWR024
 U 1 1 56620A16
 P 5550 1150
@@
 	5650 1150 5550 1150
 $Comp
-L GND #PWR025
+L GND-RESCUE-tempLoggerNG #PWR025
 U 1 1 566212ED
 P 5450 1450
@@
 $EndComp
 $Comp
-L R R5
+L R-RESCUE-tempLoggerNG R5
 U 1 1 5662131E
 P 5800 1450
@@
 $EndComp
 $Comp
-L GND #PWR026
+L GND-RESCUE-tempLoggerNG #PWR026
 U 1 1 56626314
 P 8600 4650
@@
 $EndComp
 $Comp
-L GND #PWR027
+L GND-RESCUE-tempLoggerNG #PWR027
 U 1 1 566263C1
 P 9200 4650
@@
 $EndComp
 $Comp
-L GND #PWR028
+L GND-RESCUE-tempLoggerNG #PWR028
 U 1 1 5662641D
 P 9200 6350
@@
 $EndComp
 $Comp
-L GND #PWR029
+L GND-RESCUE-tempLoggerNG #PWR029
 U 1 1 5662651B
 P 8600 6350
@@
 	9050 5300 9400 5300
 $Comp
-L GND #PWR030
+L GND-RESCUE-tempLoggerNG #PWR030
 U 1 1 56627EAA
 P 7000 4100
@@
 Connection ~ 7000 3900
 $Comp
-L GND #PWR031
+L GND-RESCUE-tempLoggerNG #PWR031
 U 1 1 566281DD
 P 10700 4100
@@
 Connection ~ 10700 3900
 $Comp
-L GND #PWR032
+L GND-RESCUE-tempLoggerNG #PWR032
 U 1 1 566285B7
 P 10700 5800
@@
 Connection ~ 10700 5600
 $Comp
-L GND #PWR033
+L GND-RESCUE-tempLoggerNG #PWR033
 U 1 1 56628A0D
 P 7000 5800
@@
 ADS_SCLK
 $Comp
-L C C8
+L C-RESCUE-tempLoggerNG C8
 U 1 1 5661C866
 P 5850 2300
@@
 Connection ~ 5850 2550
 $Comp
-L GND #PWR034
+L GND-RESCUE-tempLoggerNG #PWR034
 U 1 1 5661D3AE
 P 5850 2600
@@
 ch67_activate
 $Comp
-L R R6
+L R-RESCUE-tempLoggerNG R6
 U 1 1 56A6B163
 P 4550 4800
@@
 $EndComp
 $Comp
-L +3.3V #PWR035
+L +3.3V-RESCUE-tempLoggerNG #PWR035
 U 1 1 56A6B52D
 P 4550 4500
