File: hardware/tempLoggerNG.kicad_pcb (KiCad board)
At the start: 2 copper layers, 56.9 x 45 mm, 29 parts, among them CON1 MR-AVR-ISP-6, CON2 USB-MINI-B, IC1 ATMEGA328p, Q1 MOS_N, Q2 MOS_N, Q3 MOS_N, Q4 Q1-4: 2N7002, U1 ADS1248, U2 NCP1117-3v3, X1 12MHz

Commit message: Recover legacy KiCad symbols and migrate project to KiCad 10 format
The schematic referenced symbols (GND, R, C, +3.3V, +5V, CRYSTAL, MOS_N,
USB-MINI-B, NCP1117ST33T3G) from KiCad's pre-2013 default libraries.
Several of these had previously been rescued into a project-local cache
by an old KiCad version, but that cache was never committed, so modern
KiCad (which dropped the legacy libraries entirely) could no longer
resolve them.

Recreate the missing symbols in tempLoggerNG-rescue.lib and
localsymbols.lib using the authentic historical definitions (traced
through the kicad-library git history), validated against the actual
wire connections in the schematic. Fix an upstream duplicate-pin-number
bug in the historical NCP1117ST33T3G definition along the way.

Add sym-lib-table so the project resolves these libraries on a fresh
checkout, and commit the KiCad 10 project/schematic/PCB files produced
when re-saving in the current format. Ignore KiCad's local autosave
history directory and the now-superseded rescue-attempt artifacts.

Co-Authored-By: Claude Sonnet 5 <noreply@anthropic.com>
Other:
- net class Default removed
